Commit message: 20250427

File: Robots_usd/K188/urdf/K188.urdf (robot description, URDF)
Before this commit: robot K18, 35 links, 34 joints
Links:
- removed link pelvis
- added link base_link, mass 0.838762508448584; collision mesh filename=../meshes/base_link.STL; visual mesh filename=../meshes/base_link.STL
- added link head_link; visual sphere radius=0.0001
- added link left_hand_link; visual sphere radius=0.0001
- added link left_toe_link; visual sphere radius=0.0001
- added link right_hand_link; visual sphere radius=0.0001
- added link right_toe_link; visual sphere radius=0.0001
Joints:
- added joint headnew_joint: type fixed, parent head, child head_link, origin xyz=0 0 0.15 rpy=0 0 0
- added joint left_hand_linknew_joint: type fixed, parent left_hand, child left_hand_link, origin xyz=0 0 -0.2 rpy=0 0 0
- added joint left_toe_link_joint: type fixed, parent left_foot, child left_toe_link, origin xyz=0.15 0 0 rpy=0 0 0
- added joint right_hand_linknew_joint: type fixed, parent right_hand, child right_hand_link, origin xyz=0 0 -0.2 rpy=0 0 0
- added joint right_toe_link_joint: type fixed, parent right_foot, child right_toe_link, origin xyz=0.15 0 0 rpy=0 0 0
- joint abdomen_z: parent pelvis -> base_link
- joint left_hip_y: parent pelvis -> base_link
- joint right_hip_y: parent pelvis -> base_link
