Commit message: 20250615_cr1a_final

File: Robots_usd/CRB0/CRB0.urdf (robot description, URDF)
Before this commit: robot B-20250522, 30 links, 29 joints
Links:
- removed link body
- removed link left_ankle_x_link
- removed link left_ankle_y_link
- removed link left_elbow_link
- removed link left_hip_x_link
- removed link left_hip_y_link
- removed link left_hip_z_link
- removed link left_shoulder_x_link
- removed link left_shoulder_y_link
- removed link left_shoulder_z_link
- removed link left_wrist_x_link
- removed link left_wrist_y_link
- removed link left_wrist_z_link
- removed link right_ankle_x_link
- removed link right_ankle_y_link
- removed link right_elbow_link
- removed link right_hip_x_link
- removed link right_hip_y_link
- removed link right_hip_z_link
- removed link right_shoulder_x_link
- removed link right_shoulder_y_link
- removed link right_shoulder_z_link
- removed link right_wrist_x_link
- removed link right_wrist_y_link
- removed link right_wrist_z_link
- removed link waist_x_link
- removed link waist_z_link
- added link body_link, mass 17.72258; collision box size=0.2 0.2 0.375; collision box size=0.23 0.25 0.25
- added link left_ankle_pitch_link, mass 1.4119; collision cylinder length=0.11 radius=0.045; visual mesh filename=./meshes/ankle_y.stl
- added link left_ankle_roll_link, mass 1.78979; collision box size=0.26 0.11 0.04; visual mesh filename=./meshes/ankle_x.stl
- added link left_elbow_pitch_link, mass 2.12943; collision cylinder length=0.11 radius=0.055; collision cylinder length=0.15 radius=0.045
- added link left_hip_pitch_link, mass 1.89927; collision cylinder length=0.08 radius=0.07; collision cylinder length=0.135 radius=0.06
- added link left_hip_roll_link, mass 1.75097; collision box size=0.14 0.08 0.15; visual mesh filename=./meshes/hip_x.stl
- added link left_hip_yaw_link, mass 3.59517; collision cylinder length=0.26 radius=0.06; visual mesh filename=./meshes/hip_z.stl
- added link left_shoulder_pitch_link, mass 1.82215; collision cylinder length=0.1 radius=0.06; visual mesh filename=./meshes/shoulder_y.stl
- added link left_shoulder_roll_link, mass 0.97689; collision cylinder length=0.1 radius=0.055; collision cylinder length=0.11 radius=0.055
- added link left_shoulder_yaw_link, mass 1.9789; collision cylinder length=0.15 radius=0.055; visual mesh filename=./meshes/shoulder_z.stl
- added link left_wrist_pitch_link, mass 0.96977; collision cylinder length=0.09 radius=0.04; visual mesh filename=./meshes/wrist_y.stl
- added link left_wrist_roll_link, mass 0.31088; collision sphere radius=0.0425; visual mesh filename=./meshes/wrist_x.stl
- added link left_wrist_yaw_link, mass 0.79873; collision cylinder length=0.095 radius=0.04; visual mesh filename=./meshes/wrist_z.stl
- added link right_ankle_pitch_link, mass 1.4119; collision cylinder length=0.11 radius=0.045; visual mesh filename=./meshes/ankle_y.stl
- added link right_ankle_roll_link, mass 1.78979; collision box size=0.26 0.11 0.04; visual mesh filename=./meshes/ankle_x.stl
- added link right_elbow_pitch_link, mass 2.12943; collision cylinder length=0.11 radius=0.055; collision cylinder length=0.15 radius=0.045
- added link right_hip_pitch_link, mass 1.89927; collision cylinder length=0.08 radius=0.07; collision cylinder length=0.135 radius=0.06
- added link right_hip_roll_link, mass 1.75097; collision box size=0.14 0.08 0.15; visual mesh filename=./meshes/hip_x.stl
- added link right_hip_yaw_link, mass 3.59517; collision cylinder length=0.26 radius=0.06; visual mesh filename=./meshes/hip_z.stl
- added link right_shoulder_pitch_link, mass 1.82215; collision cylinder length=0.1 radius=0.06; visual mesh filename=./meshes/shoulder_y.stl
- added link right_shoulder_roll_link, mass 0.97689; collision cylinder length=0.1 radius=0.055; collision cylinder length=0.11 radius=0.055
- added link right_shoulder_yaw_link, mass 1.9789; collision cylinder length=0.15 radius=0.055; visual mesh filename=./meshes/shoulder_z.stl
- added link right_wrist_pitch_link, mass 0.96977; collision cylinder length=0.09 radius=0.04; visual mesh filename=./meshes/wrist_y.stl
- added link right_wrist_roll_link, mass 0.31088; collision sphere radius=0.0425; visual mesh filename=./meshes/wrist_x.stl
- added link right_wrist_yaw_link, mass 0.79873; collision cylinder length=0.095 radius=0.04; visual mesh filename=./meshes/wrist_z.stl
- added link waist_roll_link, mass 3.40004; collision box size=0.12 0.09 0.14; visual mesh filename=./meshes/waist_x.stl
- added link waist_yaw_link, mass 1.84403; collision cylinder length=0.06 radius=0.065; visual mesh filename=./meshes/waist_z.stl
Joints:
- removed joint left_ankle_x_joint
- removed joint left_ankle_y_joint
- removed joint left_elbow_joint
- removed joint left_hip_x_joint
- removed joint left_hip_y_joint
- removed joint left_hip_z_joint
- removed joint left_shoulder_x_joint
- removed joint left_shoulder_y_joint
- removed joint left_shoulder_z_joint
- removed joint left_wrist_x_joint
- removed joint left_wrist_y_joint
- removed joint left_wrist_z_joint
- removed joint right_ankle_x_joint
- removed joint right_ankle_y_joint
- removed joint right_elbow_joint
- removed joint right_hip_x_joint
- removed joint right_hip_y_joint
- removed joint right_hip_z_joint
- removed joint right_shoulder_x_joint
- removed joint right_shoulder_y_joint
- removed joint right_shoulder_z_joint
- removed joint right_wrist_x_joint
- removed joint right_wrist_y_joint
- removed joint right_wrist_z_joint
- removed joint waist_x_joint
- removed joint waist_y_joint
- removed joint waist_z_joint
- added joint left_ankle_pitch_joint: type revolute, parent left_knee_link, child left_ankle_pitch_link, origin xyz=0 0 -0.41 rpy=0 0 0, axis 0 1 0, limit lower=-1.0472 upper=0.7854 effort=107 velocity=19.38
- added joint left_ankle_roll_joint: type revolute, parent left_ankle_pitch_link, child left_ankle_roll_link, origin xyz=0 0 0 rpy=0 0 0, axis 1 0 0, limit lower=-0.61087 upper=0.61087 effort=31 velocity=23.76
- added joint left_elbow_pitch_joint: type revolute, parent left_shoulder_yaw_link, child left_elbow_pitch_link, origin xyz=0 0 0 rpy=0 -1.57079633 0, axis 0 1 0, limit lower=-0.767945 upper=1.74533 effort=107 velocity=19.38
- added joint left_hip_pitch_joint: type revolute, parent base_link, child left_hip_pitch_link, origin xyz=0 0.162 0 rpy=0 0 0, axis 0 1 0, limit lower=-2.7925 upper=1.5708 effort=413 velocity=20
- added joint left_hip_roll_joint: type revolute, parent left_hip_pitch_link, child left_hip_roll_link, origin xyz=0 0 0 rpy=0 0 0, axis 1 0 0, limit lower=-0.43633 upper=2.618 effort=107 velocity=19.38
- added joint left_hip_yaw_joint: type revolute, parent left_hip_roll_link, child left_hip_yaw_link, origin xyz=0 0 -0.142 rpy=0 0 0, axis 0 0 1, limit lower=-0.5236 upper=3.6652 effort=107 velocity=19.38
- added joint left_shoulder_pitch_joint: type revolute, parent body_link, child left_shoulder_pitch_link, origin xyz=-0.03 0.22635 0.225 rpy=0 0 0, axis 0 1 0, limit lower=-3.3161 upper=1.5708 effort=107 velocity=19.38
- added joint left_shoulder_roll_joint: type revolute, parent left_shoulder_pitch_link, child left_shoulder_roll_link, origin xyz=0 0 0 rpy=0 0 0, axis 1 0 0, limit lower=-0.43633 upper=3.5779 effort=107 velocity=19.38
- added joint left_shoulder_yaw_joint: type revolute, parent left_shoulder_roll_link, child left_shoulder_yaw_link, origin xyz=0 0 -0.265 rpy=0 0 0, axis 0 0 1, limit lower=-2.9671 upper=2.9671 effort=107 velocity=19.38
- added joint left_wrist_pitch_joint: type revolute, parent left_wrist_yaw_link, child left_wrist_pitch_link, origin xyz=0 0 0 rpy=0 0 0, axis 0 1 0, limit lower=-1.5708 upper=1.5708 effort=31 velocity=23.76
- added joint left_wrist_roll_joint: type revolute, parent left_wrist_pitch_link, child left_wrist_roll_link, origin xyz=0 0 -0.08 rpy=0 0 0, axis 1 0 0, limit lower=-1.5708 upper=1.5708 effort=31 velocity=23.76
- added joint left_wrist_yaw_joint: type revolute, parent left_elbow_pitch_link, child left_wrist_yaw_link, origin xyz=0 0 -0.16 rpy=0 0 0, axis 0 0 1, limit lower=-2.9671 upper=2.9671 effort=31 velocity=23.76
- added joint right_ankle_pitch_joint: type revolute, parent right_knee_link, child right_ankle_pitch_link, origin xyz=0 0 -0.41 rpy=0 0 0, axis 0 1 0, limit lower=-1.0472 upper=0.7854 effort=107 velocity=19.38
- added joint right_ankle_roll_joint: type revolute, parent right_ankle_pitch_link, child right_ankle_roll_link, origin xyz=0 0 0 rpy=0 0 0, axis 1 0 0, limit lower=-0.61087 upper=0.61087 effort=31 velocity=23.76
- added joint right_elbow_pitch_joint: type revolute, parent right_shoulder_yaw_link, child right_elbow_pitch_link, origin xyz=0 0 0 rpy=0 -1.57079632 0, axis 0 1 0, limit lower=-0.767945 upper=1.74533 effort=107 velocity=19.38
- added joint right_hip_pitch_joint: type revolute, parent base_link, child right_hip_pitch_link, origin xyz=0 -0.162 0 rpy=0 0 0, axis 0 1 0, limit lower=-2.7925 upper=1.5708 effort=413 velocity=20
- added joint right_hip_roll_joint: type revolute, parent right_hip_pitch_link, child right_hip_roll_link, origin xyz=0 0 0 rpy=0 0 0, axis 1 0 0, limit lower=-2.618 upper=0.43633 effort=107 velocity=19.38
- added joint right_hip_yaw_joint: type revolute, parent right_hip_roll_link, child right_hip_yaw_link, origin xyz=0 0 -0.142 rpy=0 0 0, axis 0 0 1, limit lower=-3.6652 upper=0.5236 effort=107 velocity=19.38
- added joint right_shoulder_pitch_joint: type revolute, parent body_link, child right_shoulder_pitch_link, origin xyz=-0.03 -0.22635 0.225 rpy=0 0 0, axis 0 1 0, limit lower=-3.3161 upper=1.5708 effort=107 velocity=19.38
- added joint right_shoulder_roll_joint: type revolute, parent right_shoulder_pitch_link, child right_shoulder_roll_link, origin xyz=0 0 0 rpy=0 0 0, axis 1 0 0, limit lower=-3.5779 upper=0.43633 effort=107 velocity=19.38
- added joint right_shoulder_yaw_joint: type revolute, parent right_shoulder_roll_link, child right_shoulder_yaw_link, origin xyz=0 0 -0.265 rpy=0 0 0, axis 0 0 1, limit lower=-2.9671 upper=2.9671 effort=107 velocity=19.38
- added joint right_wrist_pitch_joint: type revolute, parent right_wrist_yaw_link, child right_wrist_pitch_link, origin xyz=0 0 0 rpy=0 0 0, axis 0 1 0, limit lower=-1.5708 upper=1.5708 effort=31 velocity=23.76
- added joint right_wrist_roll_joint: type revolute, parent right_wrist_pitch_link, child right_wrist_roll_link, origin xyz=0 0 -0.08 rpy=0 0 0, axis 1 0 0, limit lower=-1.5708 upper=1.5708 effort=31 velocity=23.76
- added joint right_wrist_yaw_joint: type revolute, parent right_elbow_pitch_link, child right_wrist_yaw_link, origin xyz=0 0 -0.16 rpy=0 0 0, axis 0 0 1, limit lower=-2.9671 upper=2.9671 effort=31 velocity=23.76
- added joint waist_pitch_joint: type revolute, parent waist_roll_link, child body_link, origin xyz=0 0 0.114 rpy=0 0 0, axis 0 1 0, limit lower=-0.5236 upper=1.5708 effort=413 velocity=20
- added joint waist_roll_joint: type revolute, parent waist_yaw_link, child waist_roll_link, origin xyz=0 0 0. rpy=0 0 0, axis 1 0 0, limit lower=-0.7854 upper=0.7854 effort=107 velocity=19.38
- added joint waist_yaw_joint: type revolute, parent base_link, child waist_yaw_link, origin xyz=0 0 0.176 rpy=0 0 0, axis 0 0 1, limit lower=-3.6652 upper=1.7453 effort=107 velocity=19.38
- joint left_knee_joint: parent left_hip_z_link -> left_hip_yaw_link
- joint right_knee_joint: parent right_hip_z_link -> right_hip_yaw_link
