Commit message: 20250924

File: Robots_usd/CRB0/CRB0_21_q.urdf (robot description, URDF)
Before this commit: robot CR01B, 30 links, 29 joints
Links:
- link left_ankle_roll_link: geometry collision box size=0.18 0.12 0.04; collision sphere radius=0.035
- link right_ankle_roll_link: geometry collision box size=0.18 0.12 0.04; collision sphere radius=0.035
